File: pmod_esp32_2layer/pmod_esp32.kicad_pcb (KiCad board)
At the start: 2 copper layers, 50.4 x 24.5 mm, 27 parts, among them J1 4-Pin Male Header, Through Ho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, J2 2x6 Pin Male Header, Through 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, U1 ESP-WROOM-32, U2 TS3A5018PWR

Commit message: Some issues have been resolved
Parts:
- added G***: LOGO, Logo:kou_logo_5mm, F.Cu at (213.6, 42.1)
- added G***: LOGO, Logo:kou_logo_5mm, B.Cu at (219.6, 39.9)
- J1: footprint 68001-204HLF:AMPHENOL_68001-204HLF -> M20-9990446:HARWIN_M20-9990446
- J2: footprint m20-9740642:M209740642 -> KiCad:M209740642
- U2: footprint TS3A5018PW:SOP65P640X120-16N -> TS3A5018PWR:SOP65P640X120-16N
Routing:
- net /EN: track 47.1 -> 49.9 mm
- net /VCC3V3: track 76.6 -> 77.4 mm
Other:
- board text added: "Muhtas 1 Project 200207032 Nida Mert"

Commit message: The final versions of the PCB designs have been added.
Routing:
- net /GND: vias 179 -> 182
Changed lines of the file:
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@@
 			(at 6.885 -3.585 180)
 			(layer "B.Fab")
+			(hide yes)
 			(effects
 				(font
@@
 	)
 	(via
+		(at 206.95 43.825)
+		(size 0.6)
+		(drill 0.3)
+		(layers "F.Cu" "B.Cu")
+		(free yes)
+		(net 2)
+	)
+	(via
 		(at 237.25 51)
 		(size 0.6)
@@
 	)
 	(via
+		(at 207.8 45.4)
+		(size 0.6)
+		(drill 0.3)
+		(layers "F.Cu" "B.Cu")
+		(free yes)
+		(net 2)
+	)
+	(via
 		(at 196.45 50.2)
 		(size 0.6)
@@
 		(size 0.6)
 		(drill 0.3)
+		(layers "F.Cu" "B.Cu")
+		(free yes)
+		(net 2)
+	)
+	(via
+		(at 207.825 44.575)
+		(size 0.6)
+		(drill 0.3)
