File: pmod_esp32_2layer/pmod_esp32.kicad_sch (KiCad schematic)
At the start: 27 parts, among them J1 4-Pin Male Header, Through Ho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, J2 2x6 Pin Male Header, Through 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, U1 ESP-WROOM-32, U2 TS3A5018PWR

Commit message: Some issues have been resolved
Parts:
- J1: footprint 68001-204HLF:AMPHENOL_68001-204HLF -> HDRV4W67P0X254_1X4_1016X241X858P; Height (none) -> 8.58; Manufacturer_Name (none) -> Amphenol Communications Solutions; Manufacturer_Part_Number (none) -> 68001-204HLF
- U1: Availability In Stock -> Not in stock; Check_prices https://www.direnc.net/esp-wroom32-modul -> https://www.snapeda.com/parts/ESP-WROOM-32/Espressif+System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; Description_1 ESP-WROOM-32 series Transceiver; 802.11 b/g/n (Wi-Fi, WiFi, WLAN), Bluetooth® Smart 4.x Low Energy (BLE) Evaluation Board -> ESP-WROOM-32 series Transceiver; 802.11 b/g/n (Wi-Fi, WiFi, WLAN), Bluetooth® Smart 4.x Low Energy (BLE) Evaluation Board; Package 18±0.2mmx25.5±0.2mmx3.1±0.15mm -> Module Espressif Systems; Price 125.56 TL -> None
- U2: footprint TS3A5018PW:SOP65P640X120-16N -> TS3A5018PWR:SOP65P640X120-16N
Changed lines of the file:
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@@
 			)
 		)
-		(property "Footprint" "TS3A5018PW:SOP65P640X120-16N"
+		(property "Footprint" "TS3A5018PWR:SOP65P640X120-16N"
 			(at 227.33 50.8 0)
 			(effects
@@
 			)
 		)
-		(property "Datasheet" "https://pdf.direnc.net/upload/20-pin-2x10-2-54mm-erkek-pin-header-tht-90c-datasheet.pdf"
+		(property "Datasheet" "https://cdn.harwin.com/pdfs/M20-974.pdf"
 			(at 91.44 338.43 0)
 			(effects
@@
 			)
 		)
-		(property "Package" "18±0.2mmx25.5±0.2mmx3.1±0.15mm"
+		(property "Package" "Module Espressif Systems"
 			(at 105.41 66.04 0)
 			(effects
@@
 			)
 		)
-		(property "Check_prices" "https://www.direnc.net/esp-wroom32-modul"
+		(property "Check_prices" "https://www.snapeda.com/parts/ESP-WROOM-32/Espressif+Systems/view-part/?ref=eda"
 			(at 105.41 66.04 0)
 			(effects
@@
 			)
 		)
-		(property "Price" "125.56 TL"
+		(property "Price" "None"
 			(at 105.41 66.04 0)
 			(effects
@@
 			)
 		)
-		(property "Availability" "In Stock"
+		(property "Availability" "Not in stock"
 			(at 105.41 66.04 0)
 			(effects
@@
 			)
 		)
-		(property "Description_1" "\nESP-WROOM-32 series Transceiver; 802.11 b/g/n (Wi-Fi, WiFi, WLAN), Bluetooth® Smart 4.x Low Energy (BLE) Evaluation Board\n"
+		(property "Description_1" "\n                        \n                            ESP-WROOM-32 series Transceiver; 802.11 b/g/n (Wi-Fi, WiFi, WLAN), Bluetooth® Smart 4.x Low Energy (BLE) Evaluation Board\n                        \n"
 			(at 105.41 66.04 0)
 			(effects
@@
 	(symbol
 		(lib_id "68001-204HLF:68001-204HLF")
-		(at 36.83 181.61 0)
+		(at 29.21 179.07 0)
 		(unit 1)
 		(exclude_from_sim no)
@@
 		(on_board yes)
 		(dnp no)
-		(fields_autoplaced yes)
 		(property "Reference" "J1"
-			(at 43.18 181.6099 0)
+			(at 34.036 175.26 0)
 			(effects
 				(font
@@
 		)
 		(property "Value" "4-Pin Male Header, Through Hole"
-			(at 43.18 184.1499 0)
+			(at 34.29 190.754 0)
 			(effects
 				(font
@@
 			)
 		)
-		(property "Footprint" "68001-204HLF:AMPHENOL_68001-204HLF"
-			(at 36.83 181.61 0)
-			(effects
-				(font
-					(size 1.27 1.27)
-				)
-				(justify bottom)
-				(hide yes)
-			)
-		)
-		(property "Datasheet" "https://pdf.direnc.net/upload/5-pin-1x5-2-54mm-erkek-pin-header-tht-datasheet.pdf"
-			(at 36.83 181.61 0)
-			(effects
-				(font
-					(size 1.27 1.27)
-				)
-				(hide yes)
-			)
-		)
-		(property "Description" "5-Pin Single Row Male Header, 2.54mm Pitch, Through-Hole Mount"
-			(at 36.83 181.61 0)
+		(property "Footprint" "HDRV4W67P0X254_1X4_1016X241X858P"
+			(at 29.21 179.07 0)
+			(effects
+				(font
+					(size 1.27 1.27)
+				)
+				(justify bottom)
+				(hide yes)
+			)
+		)
+		(property "Datasheet" "https://cdn.amphenol-cs.com/media/wysiwyg/files/drawing/68000.pdf"
+			(at 29.21 179.07 0)
+			(effects
+				(font
+					(size 1.27 1.27)
+				)
+				(hide yes)
+			)
+		)
+		(property "Description" "BergStik<sup>&reg;</sup>, Board to Board connector, Unshrouded vertical header, Through Hole, Single Row, , 4  Positions, 2.54 mm (0.100in) Pitch."
+			(at 29.21 179.07 0)
 			(effects
 				(font
@@
 		)
 		(property "MF" "Amphenol"
-			(at 36.83 181.61 0)
+			(at 29.21 179.07 0)
 			(effects
 				(font
@@
 		)
 		(property "MAXIMUM_PACKAGE_HEIGHT" "11.43mm"
-			(at 36.83 181.61 0)
+			(at 29.21 179.07 0)
 			(effects
 				(font
@@
 		)
 		(property "Package" "None"
-			(at 36.83 181.61 0)
+			(at 29.21 179.07 0)
 			(effects
 				(font
@@
 		)
 		(property "Price" "6.59 TL"
-			(at 36.83 181.61 0)
+			(at 29.21 179.07 0)
 			(effects
 				(font
@@
 		)
 		(property "Check_prices" "https://www.snapeda.com/parts/68001-204HLF/Amphenol/view-part/?ref=eda"
-			(at 36.83 181.61 0)
+			(at 29.21 179.07 0)
 			(effects
 				(font
@@
 		)
 		(property "STANDARD" "Manufacturer Recommendations"
-			(at 36.83 181.61 0)
+			(at 29.21 179.07 0)
 			(effects
 				(font
@@
 		)
 		(property "PARTREV" "DG"
-			(at 36.83 181.61 0)
+			(at 29.21 179.07 0)
 			(effects
 				(font
@@
 		)
 		(property "SnapEDA_Link" "https://www.snapeda.com/parts/68001-204HLF/Amphenol/view-part/?ref=snap"
-			(at 36.83 181.61 0)
+			(at 29.21 179.07 0)
 			(effects
 				(font
@@
 		)
 		(property "MP" "68001-204HLF"
-			(at 36.83 181.61 0)
+			(at 29.21 179.07 0)
 			(effects
 				(font
@@
 		)
 		(property "Description_1" "\nConn; Rect; Header; Unshrouded; 4 Pos; 2.54mm Pitch; 1-Row; Thru-Hole; BergStik | Amphenol FCI (Amphenol CS) 68001-204HLF\n"
-			(at 36.83 181.61 0)
+			(at 29.21 179.07 0)
 			(effects
 				(font
@@
 		)
 		(property "Availability" "In Stock"
-			(at 36.83 181.61 0)
+			(at 29.21 179.07 0)
 			(effects
 				(font
@@
 		)
 		(property "MANUFACTURER" "Connfly"
-			(at 36.83 181.61 0)
+			(at 29.21 179.07 0)
 			(effects
 				(font
@@
 		)
 		(property "PACKAGE" "1x4 Pin Header, 2.54mm, Male "
-			(at 36.83 181.61 0)
-			(effects
-				(font
-					(size 1.27 1.27)
-				)
-				(hide yes)
-			)
+			(at 29.21 179.07 0)
+			(effects
+				(font
+					(size 1.27 1.27)
+				)
+				(hide yes)
+			)
+		)
+		(property "Height" "8.58"
+			(at 45.72 573.99 0)
+			(effects
+				(font
+					(size 1.27 1.27)
+				)
+				(justify left top)
+				(hide yes)
+			)
+		)
+		(property "Mouser Part Number" ""
+			(at 45.72 673.99 0)
+			(effects
+				(font
+					(size 1.27 1.27)
+				)
+				(justify left top)
+				(hide yes)
+			)
+		)
+		(property "Mouser Price/Stock" ""
+			(at 45.72 773.99 0)
+			(effects
+				(font
+					(size 1.27 1.27)
+				)
+				(justify left top)
+				(hide yes)
+			)
+		)
+		(property "Manufacturer_Name" "Amphenol Communications Solutions"
+			(at 45.72 873.99 0)
+			(effects
+				(font
+					(size 1.27 1.27)
+				)
+				(justify left top)
+				(hide yes)
+			)
+		)
+		(property "Manufacturer_Part_Number" "68001-204HLF"
+			(at 45.72 973.99 0)
+			(effects
+				(font
+					(size 1.27 1.27)
+				)
+				(justify left top)
+				(hide yes)
+			)

Commit message: The final versions of the PCB designs have been added.
Parts:
- C1, C2, C3, C4: symbol Device:C_Small -> Library:C_Small
- J1: symbol 68001-204HLF:68001-204HLF -> Library:68001-204HLF
- J2: symbol M20-9740642:M20-9740642 -> Library:M20-9740642
- LD0, LD1: symbol Device:LED -> Library:LED
- R1, R15, R16, R17, R18, R19, R2, R20, R21, R22, R3, R4, R5, R6, R7: symbol Device:R_Small -> Library:R_Small
- S1: symbol 430182050816:430182050816 -> Library:430182050816
- S2: symbol 418121270802:418121270802 -> Library:418121270802
- U1: symbol ESP-WROOM-32:ESP-WROOM-32 -> Library:ESP-WROOM-32
- U2: symbol TS3A5018PWR:TS3A5018PWR -> Library:TS3A5018PWR
Changed lines of the file:
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@@
 	)
 	(symbol
-		(lib_id "Device:LED")
+		(lib_id "Library:LED")
 		(at 203.2 105.41 270)
 		(mirror x)
@@
 	)
 	(symbol
-		(lib_id "Device:R_Small")
+		(lib_id "Library:R_Small")
 		(at 53.34 156.21 270)
 		(mirror x)
@@
 	)
 	(symbol
-		(lib_id "Device:R_Small")
+		(lib_id "Library:R_Small")
 		(at 58.42 160.02 270)
 		(mirror x)
@@
 	)
 	(symbol
-		(lib_id "Device:R_Small")
+		(lib_id "Library:R_Small")
 		(at 64.77 38.1 0)
 		(unit 1)
@@
 	)
 	(symbol
-		(lib_id "Device:R_Small")
+		(lib_id "Library:R_Small")
 		(at 52.07 143.51 270)
 		(mirror x)
@@
 	)
 	(symbol
-		(lib_id "Device:C_Small")
+		(lib_id "Library:C_Small")
 		(at 64.77 27.94 0)
 		(unit 1)
@@
 	)
 	(symbol
-		(lib_id "Device:C_Small")
+		(lib_id "Library:C_Small")
 		(at 73.66 27.94 0)
 		(unit 1)
@@
 	)
 	(symbol
-		(lib_id "Device:R_Small")
+		(lib_id "Library:R_Small")
 		(at 149.86 100.33 0)
 		(unit 1)
@@
 	)
 	(symbol
-		(lib_id "TS3A5018PWR:TS3A5018PWR")
+		(lib_id "Library:TS3A5018PWR")
 		(at 227.33 50.8 0)
 		(unit 1)
@@
 	)
 	(symbol
-		(lib_id "Device:R_Small")
+		(lib_id "Library:R_Small")
 		(at 153.67 76.2 90)
 		(unit 1)
@@
 	)
 	(symbol
-		(lib_id "Device:R_Small")
+		(lib_id "Library:R_Small")
 		(at 149.86 114.3 0)
 		(unit 1)
@@
 	)
 	(symbol
-		(lib_id "M20-9740642:M20-9740642")
+		(lib_id "Library:M20-9740642")
 		(at 72.39 143.51 0)
 		(unit 1)
@@
 	)
 	(symbol
-		(lib_id "Device:C_Small")
+		(lib_id "Library:C_Small")
 		(at 255.27 33.02 0)
 		(unit 1)
@@
 	)
 	(symbol
-		(lib_id "Device:R_Small")
+		(lib_id "Library:R_Small")
 		(at 218.44 120.65 0)
 		(unit 1)
@@
 	)
 	(symbol
-		(lib_id "Device:R_Small")
+		(lib_id "Library:R_Small")
 		(at 143.51 82.55 0)
 		(unit 1)
@@
 	)
 	(symbol
-		(lib_id "Device:R_Small")
+		(lib_id "Library:R_Small")
 		(at 111.76 148.59 90)
 		(unit 1)
@@
 	)
 	(symbol
-		(lib_id "Device:LED")
+		(lib_id "Library:LED")
 		(at 218.44 105.41 270)
 		(mirror x)
@@
 	)
 	(symbol
-		(lib_id "Device:R_Small")
+		(lib_id "Library:R_Small")
 		(at 116.84 143.51 90)
 		(unit 1)
@@
 	)
 	(symbol
-		(lib_id "ESP-WROOM-32:ESP-WROOM-32")
+		(lib_id "Library:ESP-WROOM-32")
 		(at 105.41 66.04 0)
 		(mirror y)
@@
 	)
 	(symbol
-		(lib_id "Device:R_Small")
+		(lib_id "Library:R_Small")
 		(at 57.15 148.59 270)
 		(mirror x)
@@
 	)
 	(symbol
-		(lib_id "418121270802:418121270802")
+		(lib_id "Library:418121270802")
 		(at 157.48 91.44 270)
 		(mirror x)
@@
 	)
 	(symbol
-		(lib_id "Device:R_Small")
+		(lib_id "Library:R_Small")
 		(at 203.2 120.65 0)
 		(unit 1)
@@
 	)
 	(symbol
-		(lib_id "68001-204HLF:68001-204HLF")
+		(lib_id "Library:68001-204HLF")
 		(at 29.21 179.07 0)
 		(unit 1)
@@
 	)
 	(symbol
-		(lib_id "Device:R_Small")
+		(lib_id "Library:R_Small")
 		(at 115.57 156.21 90)
 		(unit 1)
@@
 	)
 	(symbol
-		(lib_id "Device:R_Small")
+		(lib_id "Library:R_Small")
 		(at 110.49 160.02 90)
 		(unit 1)
@@
 	)
 	(symbol
-		(lib_id "Device:C_Small")
+		(lib_id "Library:C_Small")
 		(at 55.88 49.53 0)
 		(unit 1)
@@
 	)
 	(symbol
-		(lib_id "430182050816:430182050816")
+		(lib_id "Library:430182050816")
 		(at 35.56 60.96 90)
 		(unit 1)
