File: pmod_esp32_4_layer/pmod_esp32_4_layer.kicad_sch/pmod_esp32_4_layer.kicad_sch.kicad_pcb (KiCad board)
At the start: 4 copper layers, 50 x 25 mm, 27 parts, among them J1 4-Pin Male Header, Through Ho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, J2 2x6 Pin Male Header, Through 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, U1 ESP-WROOM-32, U2 TS3A5018PWR

Commit message: Some issues have been resolved
Parts:
- added G***: LOGO, Logo:kou_logo_7mm, F.Cu at (151.2, 108.0)
- added G***: LOGO, Logo:kou_logo_7mm, B.Cu at (167.9, 97.4)
Other:
- board text added: "Muhtas 1 Project 200207032 Nida Mert"

Commit message: The final versions of the PCB designs have been added.
Parts:
- moved R12 0.58 mm to (131.7, 115.2)
- moved R11 0.58 mm to (133.6, 115.2)
Changed lines of the file:
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@@
 			(outputformat 1)
 			(mirror no)
-			(drillshape 1)
+			(drillshape 0)
 			(scaleselection 1)
 			(outputdirectory "")
@@
 	(footprint "Resistor_SMD:R_0603_1608Metric_Pad0.98x0.95mm_HandSolder"
 		(layer "F.Cu")
-		(at 133.55 114.6 -90)
+		(at 133.575 115.175 -90)
 		(descr "Resistor SMD 0603 (1608 Metric), square (rectangular) end terminal, IPC_7351 nominal with elongated pad for handsoldering. (Body size source: IPC-SM-782 page 72, https://www.pcb-3d.com/wordpress/wp-content/uploads/ipc-sm-782a_amendment_1_and_2.pdf), generated with kicad-footprint-generator")
 		(tags "resistor handsolder")
 		(property "Reference" "R11"
-			(at 1.4 -1.65 180)
+			(at 1.375 -1.575 180)
 			(layer "F.SilkS")
 			(effects
@@
 		(tags "capacitor handsolder")
 		(property "Reference" "C3"
-			(at -2.3 0 0)
+			(at -2.2625 0.475 0)
 			(layer "F.SilkS")
 			(effects
@@
 	(footprint "Resistor_SMD:R_0603_1608Metric_Pad0.98x0.95mm_HandSolder"
 		(layer "F.Cu")
-		(at 131.7 114.6 90)
+		(at 131.725 115.175 90)
 		(descr "Resistor SMD 0603 (1608 Metric), square (rectangular) end terminal, IPC_7351 nominal with elongated pad for handsoldering. (Body size source: IPC-SM-782 page 72, https://www.pcb-3d.com/wordpress/wp-content/uploads/ipc-sm-782a_amendment_1_and_2.pdf), generated with kicad-footprint-generator")
 		(tags "resistor handsolder")
 		(property "Reference" "R12"
-			(at -1.4 -1.6 180)
+			(at -1.325 -1.625 180)
 			(layer "F.SilkS")
 			(effects
@@
 	)
 	(segment
+		(start 131.1125 113.65)
+		(end 131.725 114.2625)
+		(width 0.64)
+		(layer "F.Cu")
+		(net 2)
+	)
+	(segment
 		(start 144.05 100.5875)
 		(end 142.5875 100.5875)
@@
 	)
 	(segment
-		(start 130.8375 113.6875)
-		(end 131.7 113.6875)
+		(start 169.375 93.5)
+		(end 169.375 94.475)
 		(width 0.64)
 		(layer "F.Cu")
@@
 	)
 	(segment
-		(start 169.375 93.5)
-		(end 169.375 94.475)
+		(start 150.1875 103.1375)
+		(end 150.1875 101.95)
 		(width 0.64)
 		(layer "F.Cu")
@@
 	)
 	(segment
-		(start 150.1875 103.1375)
-		(end 150.1875 101.95)
+		(start 130.8 113.65)
+		(end 131.1125 113.65)
 		(width 0.64)
 		(layer "F.Cu")
@@
 	)
 	(segment
-		(start 131.7 115.5125)
-		(end 133.55 115.5125)
+		(start 141.307097 108.792903)
+		(end 141.307097 107.301471)
 		(width 0.254)
 		(layer "F.Cu")
@@
 	)
 	(segment
-		(start 141.307097 108.792903)
-		(end 141.307097 107.301471)
-		(width 0.254)
+		(start 133.575 116.0875)
+		(end 131.725 116.0875)
+		(width 0.2)
 		(layer "F.Cu")
 		(net 21)
@@
 	)
 	(segment
-		(start 134.5375 115.5125)
-		(end 134.55 115.5)
-		(width 0.254)
+		(start 133.575 116.0875)
+		(end 133.9625 116.0875)
+		(width 0.2)
 		(layer "F.Cu")
 		(net 21)
 	)
 	(segment
-		(start 133.55 115.5125)
-		(end 134.5375 115.5125)
+		(start 145.521659 107.163711)
+		(end 145.823001 106.862369)
 		(width 0.254)
 		(layer "F.Cu")
@@
 	)
 	(segment
-		(start 145.521659 107.163711)
-		(end 145.823001 106.862369)
-		(width 0.254)
+		(start 133.9625 116.0875)
+		(end 134.55 115.5)
+		(width 0.2)
 		(layer "F.Cu")
 		(net 21)
@@
 	)
 	(via
-		(at 134.55 115.5)
+		(at 138.5 111.6)
 		(size 0.6)
 		(drill 0.3)
@@
 	)
 	(via
-		(at 138.5 111.6)
+		(at 134.55 115.5)
 		(size 0.6)
 		(drill 0.3)
@@
 	)
 	(segment
-		(start 135.25 114.9)
+		(start 135.325 114.9)
 		(end 137.7275 114.9)
-		(width 0.254)
+		(width 0.2)
 		(layer "F.Cu")
 		(net 26)
 	)
 	(segment
-		(start 133.55 113.6875)
-		(end 134.0375 113.6875)
-		(width 0.254)
+		(start 133.575 114.2625)
+		(end 134.6875 114.2625)
+		(width 0.2)
 		(layer "F.Cu")
 		(net 26)
 	)
 	(segment
-		(start 134.0375 113.6875)
-		(end 135.25 114.9)
-		(width 0.254)
+		(start 134.6875 114.2625)
+		(end 135.325 114.9)
+		(width 0.2)
 		(layer "F.Cu")
 		(net 26)
@@
 		(polygon
 			(pts
-				(xy 128.15 108.2) (xy 128.8 107.25) (xy 133.15 107.25) (xy 133.9 106.2) (xy 133.9 92.3) (xy 176.9 92.3)
-				(xy 176.9 117.3) (xy 135.15 117.35) (xy 132.6 114.6) (xy 131.25 114.6) (xy 130.15 114.1) (xy 130.15 113.1)
+				(xy 128.15 108.2) (xy 128.8 107.25) (xy 133.15 107.25) (xy 133.9 106.2) (xy 133.9 92.3) (xy 175.6 92.2)
+				(xy 175.6 117.2) (xy 135.15 117.35) (xy 132.6 114.6) (xy 131.25 114.6) (xy 130.15 114.1) (xy 130.15 113.1)
 				(xy 131.15 112.55) (xy 133.25 112.55) (xy 134.25 111.9) (xy 134.25 110.45) (xy 133.25 109.7) (xy 128.9 109.7)
 				(xy 128.15 109.05)
@@
 		(polygon
 			(pts
-				(xy 128.15 110.5) (xy 128.9 109.8) (xy 133.55 109.8) (xy 133.9 109.2) (xy 133.9 92.3) (xy 176.9 92.3)
-				(xy 176.9 117.3) (xy 134.65 117.3) (xy 134.65 112.7) (xy 133.7 112.1) (xy 129.05 112.1) (xy 128.15 111.35)
+				(xy 128.15 110.5) (xy 128.9 109.8) (xy 133.55 109.8) (xy 133.9 109.2) (xy 133.9 92.3) (xy 175.55 92.375)
+				(xy 175.55 117.375) (xy 134.65 117.3) (xy 134.65 112.7) (xy 133.7 112.1) (xy 129.05 112.1) (xy 128.15 111.35)
 			)
 		)
